File: LSDTivSegG1/display.brd (EAGLE design)
At the start: 150 x 100 mm, 95 parts, among them IC1 MEGA8-P, IC2 MAX232, IC3 PCF8574P, IC4 PCF8574P, IC5 PCF8574P, IC6 PCF8574P

Commit message: fixed mirrored isp connector in display board
Connections:
- net +5V: now also SV1.2; no longer SV1.9
- net GND: now also SV1.10, SV1.4, SV1.6, SV1.8; no longer SV1.1, SV1.3, SV1.5, SV1.7
- net MISO: now also SV1.9; no longer SV1.2
- net MOSI: now also SV1.1; no longer SV1.10
- net RESET: now also SV1.5; no longer SV1.6
- net SCK: now also SV1.7; no longer SV1.4
Changed lines of the file:
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@@
 <contactref element="IC1" pad="8"/>
 <contactref element="IC1" pad="22"/>
-<contactref element="SV1" pad="7"/>
-<contactref element="SV1" pad="5"/>
-<contactref element="SV1" pad="3"/>
-<contactref element="SV1" pad="1"/>
 <contactref element="R39" pad="1"/>
 <contactref element="R38" pad="1"/>
@@
 </polygon>
 <contactref element="C7" pad="+"/>
+<contactref element="SV1" pad="4"/>
+<contactref element="SV1" pad="6"/>
+<contactref element="SV1" pad="8"/>
+<contactref element="SV1" pad="10"/>
 <wire x1="72.39" y1="54.61" x2="69.85" y2="62.23" width="0" layer="19" extent="1-1"/>
 <wire x1="68.58" y1="50.8" x2="72.39" y2="54.61" width="0" layer="19" extent="1-1"/>
@@
 <wire x1="-34.6964" y1="67.31" x2="-23.7236" y2="67.31" width="0" layer="19" extent="1-1"/>
 <wire x1="-53.34" y1="62.23" x2="-34.6964" y2="67.31" width="0" layer="19" extent="1-1"/>
-<wire x1="-63.5" y1="58.42" x2="-53.34" y2="62.23" width="0" layer="19" extent="1-1"/>
-<wire x1="-64.77" y1="64.77" x2="-63.5" y2="58.42" width="0" layer="19" extent="1-1"/>
-<wire x1="-67.31" y1="64.77" x2="-64.77" y2="64.77" width="0" layer="19" extent="1-1"/>
-<wire x1="-69.85" y1="64.77" x2="-67.31" y2="64.77" width="0" layer="19" extent="1-1"/>
-<wire x1="-72.39" y1="64.77" x2="-69.85" y2="64.77" width="0" layer="19" extent="1-1"/>
-<wire x1="-33.02" y1="88.9" x2="-34.6964" y2="67.31" width="0" layer="19" extent="1-1"/>
+<wire x1="-62.23" y1="67.31" x2="-53.34" y2="62.23" width="0" layer="19" extent="1-1"/>
+<wire x1="-64.77" y1="67.31" x2="-62.23" y2="67.31" width="0" layer="19" extent="1-1"/>
+<wire x1="-67.31" y1="67.31" x2="-64.77" y2="67.31" width="0" layer="19" extent="1-1"/>
+<wire x1="-69.85" y1="67.31" x2="-67.31" y2="67.31" width="0" layer="19" extent="1-1"/>
+<wire x1="-63.5" y1="58.42" x2="-62.23" y2="67.31" width="0" layer="19" extent="1-1"/>
+<wire x1="-63.5" y1="88.9" x2="-62.23" y2="67.31" width="0" layer="19" extent="1-1"/>
+<wire x1="-54.61" y1="88.9" x2="-63.5" y2="88.9" width="0" layer="19" extent="1-1"/>
+<wire x1="-52.07" y1="88.9" x2="-54.61" y2="88.9" width="0" layer="19" extent="1-1"/>
+<wire x1="-39.37" y1="88.9" x2="-52.07" y2="88.9" width="0" layer="19" extent="1-1"/>
+<wire x1="-33.02" y1="88.9" x2="-39.37" y2="88.9" width="0" layer="19" extent="1-1"/>
 <wire x1="-30.48" y1="88.9" x2="-33.02" y2="88.9" width="0" layer="19" extent="1-1"/>
 <wire x1="-27.94" y1="88.9" x2="-30.48" y2="88.9" width="0" layer="19" extent="1-1"/>
-<wire x1="-39.37" y1="88.9" x2="-33.02" y2="88.9" width="0" layer="19" extent="1-1"/>
 <wire x1="-15.24" y1="88.9" x2="-27.94" y2="88.9" width="0" layer="19" extent="1-1"/>
-<wire x1="-52.07" y1="88.9" x2="-39.37" y2="88.9" width="0" layer="19" extent="1-1"/>
-<wire x1="-54.61" y1="88.9" x2="-52.07" y2="88.9" width="0" layer="19" extent="1-1"/>
-<wire x1="-63.5" y1="88.9" x2="-54.61" y2="88.9" width="0" layer="19" extent="1-1"/>
 <wire x1="-76.2" y1="88.9" x2="-63.5" y2="88.9" width="0" layer="19" extent="1-1"/>
 <wire x1="-81.28" y1="88.9" x2="-76.2" y2="88.9" width="0" layer="19" extent="1-1"/>
@@
 <wire x1="-121.92" y1="124.46" x2="-127" y2="96.52" width="0" layer="19" extent="1-1"/>
 <wire x1="-102.87" y1="130.81" x2="-121.92" y2="124.46" width="0" layer="19" extent="1-1"/>
-<wire x1="-101.6" y1="58.42" x2="-72.39" y2="64.77" width="0" layer="19" extent="1-1"/>
+<wire x1="-101.6" y1="58.42" x2="-100.33" y2="88.9" width="0" layer="19" extent="1-1"/>
 </signal>
 <signal name="RESET">
@@
 <contactref element="R1" pad="1"/>
 <contactref element="C1" pad="1"/>
-<contactref element="SV1" pad="6"/>
+<contactref element="SV1" pad="5"/>
 <wire x1="50.8" y1="54.61" x2="54.61" y2="54.61" width="0" layer="19" extent="1-1"/>
 <wire x1="54.61" y1="50.8" x2="54.61" y2="54.61" width="0" layer="19" extent="1-1"/>
-<wire x1="-67.31" y1="67.31" x2="50.8" y2="54.61" width="0" layer="19" extent="1-1"/>
+<wire x1="-67.31" y1="64.77" x2="50.8" y2="54.61" width="0" layer="19" extent="1-1"/>
 </signal>
 <signal name="+5V">
@@
 <contactref element="IC1" pad="7"/>
 <contactref element="C8" pad="1"/>
-<contactref element="SV1" pad="9"/>
 <contactref element="R10" pad="2"/>
 <contactref element="R11" pad="2"/>
@@
 <contactref element="IC6" pad="1"/>
 <contactref element="JP1" pad="2"/>
+<contactref element="SV1" pad="2"/>
 <wire x1="72.39" y1="62.23" x2="74.93" y2="62.23" width="0" layer="19" extent="1-1"/>
 <wire x1="69.85" y1="54.61" x2="72.39" y2="62.23" width="0" layer="19" extent="1-1"/>
@@
 <wire x1="-78.74" y1="88.9" x2="-57.15" y2="88.9" width="0" layer="19" extent="1-1"/>
 <wire x1="-81.28" y1="96.52" x2="-78.74" y2="88.9" width="0" layer="19" extent="1-1"/>
+<wire x1="-72.39" y1="67.31" x2="-78.74" y2="88.9" width="0" layer="19" extent="1-1"/>
 <wire x1="-102.87" y1="88.9" x2="-81.28" y2="96.52" width="0" layer="19" extent="1-1"/>
 <wire x1="-105.41" y1="88.9" x2="-102.87" y2="88.9" width="0" layer="19" extent="1-1"/>
 <wire x1="-105.41" y1="96.52" x2="-105.41" y2="88.9" width="0" layer="19" extent="1-1"/>
-<wire x1="-62.23" y1="64.77" x2="-57.15" y2="88.9" width="0" layer="19" extent="1-1"/>
+<wire x1="-99.06" y1="58.42" x2="-72.39" y2="67.31" width="0" layer="19" extent="1-1"/>
 <wire x1="-110.49" y1="124.46" x2="-105.41" y2="96.52" width="0" layer="19" extent="1-1"/>
 <wire x1="-113.03" y1="130.81" x2="-110.49" y2="124.46" width="0" layer="19" extent="1-1"/>
@@
 <wire x1="-124.46" y1="137.16" x2="-124.46" y2="142.24" width="0" layer="19" extent="1-1"/>
 <wire x1="-133.35" y1="130.81" x2="-124.46" y2="137.16" width="0" layer="19" extent="1-1"/>
-<wire x1="-99.06" y1="58.42" x2="-102.87" y2="88.9" width="0" layer="19" extent="1-1"/>
 <wire x1="-130.81" y1="-5.08" x2="-99.06" y2="58.42" width="0" layer="19" extent="1-1"/>
 </signal>
@@
 <signal name="SCK">
 <contactref element="IC1" pad="19"/>
-<contactref element="SV1" pad="4"/>
-<wire x1="-69.85" y1="67.31" x2="77.47" y2="62.23" width="0" layer="19" extent="1-1"/>
+<contactref element="SV1" pad="7"/>
+<wire x1="-64.77" y1="64.77" x2="77.47" y2="62.23" width="0" layer="19" extent="1-1"/>
 </signal>
 <signal name="MISO">
 <contactref element="IC1" pad="18"/>
-<contactref element="SV1" pad="2"/>
-<wire x1="-72.39" y1="67.31" x2="80.01" y2="62.23" width="0" layer="19" extent="1-1"/>
+<contactref element="SV1" pad="9"/>
+<wire x1="-62.23" y1="64.77" x2="80.01" y2="62.23" width="0" layer="19" extent="1-1"/>
 </signal>
 <signal name="MOSI">
 <contactref element="IC1" pad="17"/>
-<contactref element="SV1" pad="10"/>
-<wire x1="-62.23" y1="67.31" x2="82.55" y2="62.23" width="0" layer="19" extent="1-1"/>
+<contactref element="SV1" pad="1"/>
+<wire x1="-72.39" y1="64.77" x2="82.55" y2="62.23" width="0" layer="19" extent="1-1"/>
 </signal>
 <signal name="RXD">
