File: LSDTivSegG1/display.brd (EAGLE design)
At the start: 150 x 100 mm, 99 parts, among them IC1 MEGA8-P, IC2 MAX232, IC3 PCF8574P, IC4 PCF8574P, IC5 PCF8574P, IC6 PCF8574P

Commit message: fixed some bugs in schematic board file with all components placed
Parts:
- moved C11 276.0 mm to (118.1, 74.9), turned to 270 degrees
- moved C13 273.4 mm to (129.5, 8.89)
- moved LED19 255.4 mm to (127.0, 66.0), turned to 180 degrees
- moved R32 253.5 mm to (101.6, 38.1), turned to 270 degrees
- moved IC6 245.8 mm to (137.2, 16.5), flipped to the bottom, turned to 180 degrees
- moved R31 242.0 mm to (99.1, 38.1), turned to 270 degrees
- moved LED18 234.9 mm to (119.4, 68.6), turned to 270 degrees
- moved R30 230.6 mm to (96.5, 38.1), turned to 270 degrees
- moved JP2 228.3 mm to (73.7, 80.0)
- moved R5 227.3 mm to (82.5, 24.1)
- moved R6 226.2 mm to (92.7, 82.5), turned to 270 degrees
- moved LED24 222.3 mm to (129.5, 27.9), turned to 180 degrees
- moved U$1 221.2 mm to (113.0, 5.08), turned to 180 degrees
- moved R9 221.0 mm to (141.0, 7.62), turned to 180 degrees
- moved JP1 220.3 mm to (73.7, 73.7), turned to 90 degrees
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Connections:
- net +5V: no longer R12.2, R13.2, R14.2, R15.2, R16.2, R17.2, R18.2, R19.2, R2.A, R20.2, R21.2, R22.2, R23.2, R24.2, R25.2, R26.2, R27.2, R28.2, R29.2, R30.2, R31.2, R32.2, R33.2, R34.2, R35.2, U$1.1, U$1.16
- net GND: now also R12.2, R13.2, R14.2, R15.2, R16.2, R17.2, R18.2, R19.2, R2.A, R20.2, R21.2, R22.2, R23.2, R24.2, R25.2, R26.2, R27.2, R28.2, R29.2, R30.2, R31.2, R32.2, R33.2, R34.2, R35.2, U$1.1, U$1.16
Routing:
- added copper zone on layer 16, net GND
- removed copper zone on layer 1, net GND

Commit message: working on display.brd
Parts:
- moved C7 112.0 mm to (121.9, 83.8), turned to 270 degrees
- moved C5 111.8 mm to (121.9, 78.1), turned to 90 degrees
- moved C11 92.7 mm to (26.0, 85.7), turned to 180 degrees
- moved IC2 89.5 mm to (108.6, 81.9), turned to 0 degrees
- moved C4 85.8 mm to (95.2, 78.1)
- moved C6 77.3 mm to (95.2, 83.8)
- moved R6 69.9 mm to (22.9, 83.2), turned to 0 degrees
- moved IC3 66.1 mm to (39.4, 81.9), turned to 0 degrees
- moved R10 12.1 mm to (147.3, 80.6), turned to 270 degrees
- moved R9 10.3 mm to (130.8, 5.71), turned to 0 degrees
- moved R11 9.94 mm to (147.3, 93.3), turned to 90 degrees
- moved C2 2.29 mm to (126.4, 78.7), turned to 90 degrees
- moved C3 2.29 mm to (126.4, 73.7), turned to 90 degrees
- moved C8 0.63 mm to (131.4, 82.5)
- turned LED13 to 90 degrees
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Routing:
- net +5V: track 0.00 -> 159.8 mm
- net EN: track 0.00 -> 85.7 mm, vias 0 -> 1
- net RW: track 0.00 -> 82.1 mm, vias 0 -> 1
- net RS: track 0.00 -> 78.5 mm, vias 0 -> 1
- net RESET: track 0.00 -> 71.2 mm
- net RS232TX: track 0.00 -> 50.5 mm
- net N$34: track 0.00 -> 39.4 mm
- net N$22: track 0.00 -> 39.4 mm
- net RS232RX: track 0.00 -> 39.1 mm
- net N$35: track 0.00 -> 36.9 mm
- net N$23: track 0.00 -> 36.9 mm
- net N$21: track 0.00 -> 35.4 mm
- net N$33: track 0.00 -> 35.4 mm
- net N$32: track 0.00 -> 32.5 mm
- net N$20: track 0.00 -> 32.5 mm
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