File: LSDTivSegG1/leistung.sch (EAGLE design)
At the start: 80 parts, among them IC1 LM 2576 T5,0, IC2 IR2184D, IC3 IR2184D, IC4 4081N, IC5 4069N, IC6 LM 2576 T15, IC7 IR2184D, IC8 IR2184D, IC9 TINY13-20PU, X1 057-010-1, X2 MKDSN1,5/2-5,08

Commit message: Nachbesprechung Änderungen gemacht
Parts:
- added C19, C20: 4m7, rcl:CPOL-EUE7.5-18
- added R11, R12, R13, R25: 470k, rcl:R-EU_0207/7
- C1, C11: value 10u -> 4m7; device rcl:CPOL-EUE2.5-5 -> rcl:CPOL-EUE7.5-18
- D1, D13, D14, D2: value 1N4001 -> 1N4002
- D15, D16, D17, D18, D3, D4, D5, D6: value 18 -> ZD-5W_18V
- D7, D8: value 1N 5711 -> 1N5822
- Q1, Q10, Q11, Q12, Q2, Q3, Q4, Q9: value (none) -> IRFB3077
- R10: value (none) -> 20k
Connections:
- removed net BAT_PWM_IN: IC9.PB0/PCINT0/AIN0/OC0A/MOSI
- removed net DIRL_IN_INV: IC5A.O
- removed net DIRR_IN_INV: IC5B.O
- removed net MOTOR_L_ACTIVE: IC2.!SD, IC3.!SD, IC4A.O
- removed net MOTOR_R_ACTIVE: IC4B.O, IC7.!SD, IC8.!SD
- removed net N$15: IC4C.O
- removed net N$16: IC4D.O
- removed net N$21: IC4C.I0
- removed net N$22: IC4C.I1
- removed net N$23: IC4D.I0
- removed net N$24: IC4D.I1
- removed net N$29: D16.C, Q10.G, R18.2, R23.1
- new net IN_L: IC2.IN, IC4B.O
- new net IN_L_INVD: IC3.IN, IC4D.O
- new net IN_R: IC4A.O, IC7.IN
- new net IN_R_INVD: IC4C.O, IC8.IN
- new net N$13: D16.C, Q10.G, R18.2, R23.2
- net BAT_+: now also C19.+, C20.+
- net BAT_PWM: now also IC9.PB0/PCINT0/AIN0/OC0A/MOSI
- net DIRL: now also IC4B.I0, IC5B.I; no longer IC2.IN, IC5A.I
- net DIRL_INV: now also IC4D.I0, IC5B.O; no longer IC3.IN
- net DIRR: now also IC4A.I0, IC5A.I; no longer IC5B.I, IC7.IN
- net DIRR_INV: now also IC4C.I0, IC5A.O; no longer IC8.IN
- net ENABLE: now also IC2.!SD, IC3.!SD, IC7.!SD, IC8.!SD, R11.2, R12.2, R13.2, R25.2; no longer IC4A.I0, IC4B.I0
- net GND: now also C19.-, C20.-, D16.A, D17.A, D4.A, D5.A, R11.1, R12.1, R13.1, R22.1, R23.1, R25.1, R6.1, R7.1
- net MOTOR_L_+: no longer D4.A, R7.2
- net MOTOR_L_-: no longer D5.A, R6.2
- net MOTOR_PWM_L: now also IC4B.I1, IC4D.I1; no longer IC4A.I1
- net MOTOR_PWM_R: now also IC4A.I1, IC4C.I1; no longer IC4B.I1
- net MOTOR_R_+: no longer D16.A, R23.2
- net MOTOR_R_-: no longer D17.A, R22.2
- net N$32: now also R22.2; no longer R22.1
- net N$5: now also R7.2; no longer R7.1
- net N$8: now also R6.2; no longer R6.1
Other:
- note removed: "Mosfets IRFB3077"
- note removed: "_CTL indicates position on LOW-Voltage Side of board"
- moved on the sheet: C1, C11, D16, D17, D4, D5, R18, R19, R2, R22, R23, R3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
