File: LSDTivSegG1/leistung.sch (EAGLE design)
At the start: 86 parts, among them IC1 LM 2576 T5,0, IC2 IR2184D, IC3 IR2184D, IC4 4081N, IC5 4069N, IC6 LM 2576 T15, IC7 IR2184D, IC8 IR2184D, IC9 TINY13-20PU, Q1 IRFB3077, Q10 IRFB3077, Q11 IRFB3077, Q12 IRFB3077, Q2 IRFB3077, Q3 IRFB3077, Q4 IRFB3077, Q9 IRFB3077, X1 057-010-1, X2 MKDSN1,5/2-5,08

Commit message: finalized board
Parts:
- removed IC1: LM 2576 T5,0, LM2576:LM2576-T05A
- removed IC6: LM 2576 T15, LM2576:LM2576-T05A
- added IC10: LM 2576 T15, LM2576:LM2576-T05D
- added IC11: LM 2576 T5.0, LM2576:LM2576-T05D
Connections:
- net +15V: now also IC10.FB; no longer IC6.FB
- net +24V: now also IC10.+V_IN, IC11.+V_IN; no longer IC1.+V_IN, IC6.+V_IN
- net +5V: now also IC11.FB; no longer IC1.FB
- net GND: now also IC10.GND, IC10._EN/DIS, IC11.GND, IC11._EN/DIS; no longer IC1.GND, IC1._EN/DIS, IC6.GND, IC6._EN/DIS
- net N$1: now also IC11.+V_OUT; no longer IC1.+V_OUT
- net N$4: now also IC10.+V_OUT; no longer IC6.+V_OUT
Changed lines of the file:
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@@
 <part name="P+2" library="hcontrol" deviceset="+5V" device=""/>
 <part name="GND2" library="SparkFun-Aesthetics" deviceset="GND" device=""/>
-<part name="IC1" library="LM2576" deviceset="LM2576-T05A" device="" value="LM 2576 T5,0"/>
 <part name="L1" library="rcl" deviceset="L-EU" device="0207/10" value="100u"/>
 <part name="GND3" library="supply1" deviceset="GND" device=""/>
@@
 <part name="R14" library="rcl" deviceset="R-EU_" device="0207/10" value="100"/>
 <part name="FRAME2" library="frames" deviceset="FRAME_A_L" device=""/>
-<part name="IC6" library="LM2576" deviceset="LM2576-T05A" device="" value="LM 2576 T15 "/>
 <part name="D8" library="diode" deviceset="SCHOTTKY-DIODE" device="CB429-15" value="1N5822"/>
 <part name="C8" library="rcl" deviceset="CPOL-EU" device="E2.5-7" value="100u"/>
@@
 <part name="C9" library="rcl" library_urn="urn:adsk.eagle:library:334" deviceset="CPOL-EU" device="E5-13" package3d_urn="urn:adsk.eagle:package:23375/1" value="1000u"/>
 <part name="C6" library="rcl" library_urn="urn:adsk.eagle:library:334" deviceset="CPOL-EU" device="E5-13" package3d_urn="urn:adsk.eagle:package:23375/1" value="1000u"/>
+<part name="IC10" library="LM2576" deviceset="LM2576-T05D" device="" value="LM 2576 T15"/>
+<part name="IC11" library="LM2576" deviceset="LM2576-T05D" device="" value="LM 2576 T5.0"/>
 </parts>
 <sheets>
@@
 </plain>
 <instances>
-<instance part="IC1" gate="G$1" x="119.38" y="106.68"/>
 <instance part="L1" gate="G$1" x="154.94" y="114.3" rot="R90"/>
 <instance part="GND3" gate="1" x="119.38" y="86.36"/>
@@
 <instance part="FRAME2" gate="G$2" x="172.72" y="0"/>
 <instance part="C6" gate="G$1" x="162.56" y="99.06"/>
+<instance part="IC11" gate="G$1" x="119.38" y="106.68"/>
 </instances>
 <busses>
@@
 <net name="GND" class="0">
 <segment>
-<pinref part="IC1" gate="G$1" pin="GND"/>
-<pinref part="GND3" gate="1" pin="GND"/>
-</segment>
-<segment>
 <pinref part="GND5" gate="1" pin="GND"/>
 <pinref part="D7" gate="G$1" pin="A"/>
@@
 <segment>
 <pinref part="GND10" gate="1" pin="GND"/>
-<pinref part="IC1" gate="G$1" pin="_EN/DIS"/>
 <wire x1="96.52" y1="88.9" x2="96.52" y2="104.14" width="0.1524" layer="91"/>
+<pinref part="IC11" gate="G$1" pin="_EN/DIS"/>
 </segment>
 <segment>
@@
 <wire x1="162.56" y1="93.98" x2="162.56" y2="88.9" width="0.1524" layer="91"/>
 </segment>
+<segment>
+<pinref part="GND3" gate="1" pin="GND"/>
+<pinref part="IC11" gate="G$1" pin="GND"/>
+</segment>
 </net>
 <net name="+24V" class="0">
@@
 <pinref part="P+3" gate="1" pin="+24V"/>
 <wire x1="86.36" y1="116.84" x2="86.36" y2="114.3" width="0.1524" layer="91"/>
-<pinref part="IC1" gate="G$1" pin="+V_IN"/>
 <wire x1="86.36" y1="114.3" x2="88.9" y2="114.3" width="0.1524" layer="91"/>
 <pinref part="C7" gate="G$1" pin="+"/>
@@
 <wire x1="88.9" y1="104.14" x2="88.9" y2="114.3" width="0.1524" layer="91"/>
 <junction x="88.9" y="114.3"/>
+<pinref part="IC11" gate="G$1" pin="+V_IN"/>
 </segment>
 </net>
@@
 <wire x1="172.72" y1="114.3" x2="172.72" y2="111.76" width="0.1524" layer="91"/>
 <junction x="172.72" y="114.3"/>
-<pinref part="IC1" gate="G$1" pin="FB"/>
 <wire x1="142.24" y1="104.14" x2="142.24" y2="109.22" width="0.1524" layer="91"/>
 <wire x1="142.24" y1="109.22" x2="160.02" y2="109.22" width="0.1524" layer="91"/>
@@
 <wire x1="162.56" y1="101.6" x2="162.56" y2="114.3" width="0.1524" layer="91"/>
 <junction x="162.56" y="114.3"/>
+<pinref part="IC11" gate="G$1" pin="FB"/>
 </segment>
 </net>
 <net name="N$1" class="0">
 <segment>
-<pinref part="IC1" gate="G$1" pin="+V_OUT"/>
 <pinref part="L1" gate="G$1" pin="1"/>
 <wire x1="142.24" y1="114.3" x2="147.32" y2="114.3" width="0.1524" layer="91"/>
@@
 <wire x1="147.32" y1="104.14" x2="147.32" y2="114.3" width="0.1524" layer="91"/>
 <junction x="147.32" y="114.3"/>
+<pinref part="IC11" gate="G$1" pin="+V_OUT"/>
 </segment>
 </net>
@@
 </plain>
 <instances>
-<instance part="IC6" gate="G$1" x="114.3" y="109.22"/>
 <instance part="D8" gate="G$1" x="144.78" y="104.14" rot="R90"/>
 <instance part="C8" gate="G$1" x="83.82" y="104.14"/>
@@
 <instance part="FRAME6" gate="G$2" x="172.72" y="0"/>
 <instance part="C9" gate="G$1" x="160.02" y="101.6"/>
+<instance part="IC10" gate="G$1" x="114.3" y="109.22"/>
 </instances>
 <busses>
@@
 </segment>
 <segment>
-<pinref part="IC6" gate="G$1" pin="GND"/>
-<pinref part="GND11" gate="1" pin="GND"/>
-</segment>
-<segment>
 <pinref part="GND8" gate="1" pin="GND"/>
 <pinref part="C9" gate="G$1" pin="-"/>
@@
 </segment>
 <segment>
-<pinref part="IC6" gate="G$1" pin="_EN/DIS"/>
 <pinref part="GND12" gate="1" pin="GND"/>
 <wire x1="91.44" y1="106.68" x2="91.44" y2="91.44" width="0.1524" layer="91"/>
+<pinref part="IC10" gate="G$1" pin="_EN/DIS"/>
 </segment>
 <segment>
@@
 <wire x1="170.18" y1="91.44" x2="170.18" y2="93.98" width="0.1524" layer="91"/>
 </segment>
+<segment>
+<pinref part="GND11" gate="1" pin="GND"/>
+<pinref part="IC10" gate="G$1" pin="GND"/>
+</segment>
 </net>
 <net name="+24V" class="0">
@@
 <pinref part="P+5" gate="1" pin="+24V"/>
 <wire x1="81.28" y1="116.84" x2="81.28" y2="119.38" width="0.1524" layer="91"/>
-<pinref part="IC6" gate="G$1" pin="+V_IN"/>
 <wire x1="81.28" y1="116.84" x2="83.82" y2="116.84" width="0.1524" layer="91"/>
 <pinref part="C8" gate="G$1" pin="+"/>
@@
 <wire x1="83.82" y1="106.68" x2="83.82" y2="116.84" width="0.1524" layer="91"/>
 <junction x="83.82" y="116.84"/>
+<pinref part="IC10" gate="G$1" pin="+V_IN"/>
 </segment>
 </net>
@@
 <wire x1="160.02" y1="116.84" x2="160.02" y2="109.22" width="0.1524" layer="91"/>
 <junction x="160.02" y="116.84"/>
-<pinref part="IC6" gate="G$1" pin="FB"/>
 <wire x1="137.16" y1="106.68" x2="137.16" y2="111.76" width="0.1524" layer="91"/>
 <wire x1="137.16" y1="111.76" x2="157.48" y2="111.76" width="0.1524" layer="91"/>
@@
 <wire x1="160.02" y1="104.14" x2="160.02" y2="106.68" width="0.1524" layer="91"/>
 <wire x1="160.02" y1="106.68" x2="160.02" y2="109.22" width="0.1524" layer="91"/>
+<pinref part="IC10" gate="G$1" pin="FB"/>
 </segment>
 </net>
 <net name="N$4" class="0">
 <segment>
-<pinref part="IC6" gate="G$1" pin="+V_OUT"/>
 <wire x1="137.16" y1="116.84" x2="144.78" y2="116.84" width="0.1524" layer="91"/>
 <pinref part="D8" gate="G$1" pin="C"/>
@@
 <wire x1="144.78" y1="116.84" x2="147.32" y2="116.84" width="0.1524" layer="91"/>
 <junction x="144.78" y="116.84"/>
-</segment>
-</net>
+<pinref part="IC10" gate="G$1" pin="+V_OUT"/>
+</segment>
+</net>

Commit message: added Text
Parts:
- F1, F2, F3: value (none) -> 1A
Changed lines of the file:
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@@
 <grid distance="0.1" unitdist="inch" unit="inch" style="lines" multiple="1" display="no" altdistance="0.01" altunitdist="inch" altunit="inch"/>
 <layers>
-<layer number="1" name="Top" color="4" fill="1" visible="yes" active="no"/>
-<layer number="2" name="Route2" color="16" fill="1" visible="yes" active="no"/>
-<layer number="3" name="Route3" color="17" fill="1" visible="yes" active="no"/>
-<layer number="4" name="Route4" color="18" fill="1" visible="yes" active="no"/>
-<layer number="5" name="Route5" color="19" fill="1" visible="yes" active="no"/>
-<layer number="6" name="Route6" color="25" fill="1" visible="yes" active="no"/>
-<layer number="7" name="Route7" color="26" fill="1" visible="yes" active="no"/>
-<layer number="8" name="Route8" color="27" fill="1" visible="yes" active="no"/>
-<layer number="9" name="Route9" color="28" fill="1" visible="yes" active="no"/>
-<layer number="10" name="Route10" color="29" fill="1" visible="yes" active="no"/>
-<layer number="11" name="Route11" color="30" fill="1" visible="yes" active="no"/>
-<layer number="12" name="Route12" color="20" fill="1" visible="yes" active="no"/>
-<layer number="13" name="Route13" color="21" fill="1" visible="yes" active="no"/>
-<layer number="14" name="Route14" color="22" fill="1" visible="yes" active="no"/>
-<layer number="15" name="Route15" color="23" fill="1" visible="yes" active="no"/>
-<layer number="16" name="Bottom" color="1" fill="1" visible="yes" active="no"/>
-<layer number="17" name="Pads" color="2" fill="1" visible="yes" active="no"/>
-<layer number="18" name="Vias" color="2" fill="1" visible="yes" active="no"/>
-<layer number="19" name="Unrouted" color="6" fill="1" visible="yes" active="no"/>
-<layer number="20" name="Dimension" color="24" fill="1" visible="yes" active="no"/>
-<layer number="21" name="tPlace" color="7" fill="1" visible="yes" active="no"/>
-<layer number="22" name="bPlace" color="7" fill="1" visible="yes" active="no"/>
-<layer number="23" name="tOrigins" color="15" fill="1" visible="yes" active="no"/>
-<layer number="24" name="bOrigins" color="15" fill="1" visible="yes" active="no"/>
-<layer number="25" name="tNames" color="7" fill="1" visible="yes" active="no"/>
-<layer number="26" name="bNames" color="7" fill="1" visible="yes" active="no"/>
-<layer number="27" name="tValues" color="7" fill="1" visible="yes" active="no"/>
-<layer number="28" name="bValues" color="7" fill="1" visible="yes" active="no"/>
+<layer number="1" name="Top" color="4" fill="1" visible="no" active="no"/>
+<layer number="2" name="Route2" color="16" fill="1" visible="no" active="no"/>
+<layer number="3" name="Route3" color="17" fill="1" visible="no" active="no"/>
+<layer number="4" name="Route4" color="18" fill="1" visible="no" active="no"/>
+<layer number="5" name="Route5" color="19" fill="1" visible="no" active="no"/>
+<layer number="6" name="Route6" color="25" fill="1" visible="no" active="no"/>
+<layer number="7" name="Route7" color="26" fill="1" visible="no" active="no"/>
+<layer number="8" name="Route8" color="27" fill="1" visible="no" active="no"/>
+<layer number="9" name="Route9" color="28" fill="1" visible="no" active="no"/>
+<layer number="10" name="Route10" color="29" fill="1" visible="no" active="no"/>
+<layer number="11" name="Route11" color="30" fill="1" visible="no" active="no"/>
+<layer number="12" name="Route12" color="20" fill="1" visible="no" active="no"/>
+<layer number="13" name="Route13" color="21" fill="1" visible="no" active="no"/>
+<layer number="14" name="Route14" color="22" fill="1" visible="no" active="no"/>
+<layer number="15" name="Route15" color="23" fill="1" visible="no" active="no"/>
+<layer number="16" name="Bottom" color="1" fill="1" visible="no" active="no"/>
+<layer number="17" name="Pads" color="2" fill="1" visible="no" active="no"/>
+<layer number="18" name="Vias" color="2" fill="1" visible="no" active="no"/>
+<layer number="19" name="Unrouted" color="6" fill="1" visible="no" active="no"/>
+<layer number="20" name="Dimension" color="24" fill="1" visible="no" active="no"/>
+<layer number="21" name="tPlace" color="7" fill="1" visible="no" active="no"/>
+<layer number="22" name="bPlace" color="7" fill="1" visible="no" active="no"/>
+<layer number="23" name="tOrigins" color="15" fill="1" visible="no" active="no"/>
+<layer number="24" name="bOrigins" color="15" fill="1" visible="no" active="no"/>
+<layer number="25" name="tNames" color="7" fill="1" visible="no" active="no"/>
+<layer number="26" name="bNames" color="7" fill="1" visible="no" active="no"/>
+<layer number="27" name="tValues" color="7" fill="1" visible="no" active="no"/>
+<layer number="28" name="bValues" color="7" fill="1" visible="no" active="no"/>
 <layer number="29" name="tStop" color="7" fill="3" visible="no" active="no"/>
 <layer number="30" name="bStop" color="7" fill="6" visible="no" active="no"/>
@@
 <layer number="35" name="tGlue" color="7" fill="4" visible="no" active="no"/>
 <layer number="36" name="bGlue" color="7" fill="5" visible="no" active="no"/>
-<layer number="37" name="tTest" color="7" fill="1" visible="yes" active="no"/>
-<layer number="38" name="bTest" color="7" fill="1" visible="yes" active="no"/>
+<layer number="37" name="tTest" color="7" fill="1" visible="no" active="no"/>
+<layer number="38" name="bTest" color="7" fill="1" visible="no" active="no"/>
 <layer number="39" name="tKeepout" color="4" fill="11" visible="no" active="no"/>
 <layer number="40" name="bKeepout" color="1" fill="11" visible="no" active="no"/>
@@
 <layer number="44" name="Drills" color="7" fill="1" visible="no" active="no"/>
 <layer number="45" name="Holes" color="7" fill="1" visible="no" active="no"/>
-<layer number="46" name="Milling" color="3" fill="1" visible="yes" active="no"/>
-<layer number="47" name="Measures" color="7" fill="1" visible="yes" active="no"/>
-<layer number="48" name="Document" color="7" fill="1" visible="yes" active="no"/>
-<layer number="49" name="Reference" color="7" fill="1" visible="yes" active="no"/>
-<layer number="50" name="dxf" color="7" fill="1" visible="yes" active="no"/>
-<layer number="51" name="tDocu" color="7" fill="1" visible="yes" active="no"/>
-<layer number="52" name="bDocu" color="7" fill="1" visible="yes" active="no"/>
-<layer number="53" name="tGND_GNDA" color="7" fill="9" visible="yes" active="no"/>
-<layer number="54" name="bGND_GNDA" color="1" fill="9" visible="yes" active="no"/>
-<layer number="56" name="wert" color="7" fill="1" visible="yes" active="no"/>
+<layer number="46" name="Milling" color="3" fill="1" visible="no" active="no"/>
+<layer number="47" name="Measures" color="7" fill="1" visible="no" active="no"/>
+<layer number="48" name="Document" color="7" fill="1" visible="no" active="no"/>
+<layer number="49" name="Reference" color="7" fill="1" visible="no" active="no"/>
+<layer number="50" name="dxf" color="7" fill="1" visible="no" active="no"/>
+<layer number="51" name="tDocu" color="7" fill="1" visible="no" active="no"/>
+<layer number="52" name="bDocu" color="7" fill="1" visible="no" active="no"/>
+<layer number="53" name="tGND_GNDA" color="7" fill="9" visible="no" active="no"/>
+<layer number="54" name="bGND_GNDA" color="1" fill="9" visible="no" active="no"/>
+<layer number="56" name="wert" color="7" fill="1" visible="no" active="no"/>
 <layer number="88" name="SimResults" color="9" fill="1" visible="yes" active="yes"/>
 <layer number="89" name="SimProbes" color="9" fill="1" visible="yes" active="yes"/>
@@
 <part name="IC4" library="40xx" library_urn="urn:adsk.eagle:library:80" deviceset="4081" device="N" package3d_urn="urn:adsk.eagle:package:820/2"/>
 <part name="IC5" library="40xx" library_urn="urn:adsk.eagle:library:80" deviceset="4069" device="N" package3d_urn="urn:adsk.eagle:package:820/2"/>
-<part name="F1" library="special" library_urn="urn:adsk.eagle:library:367" deviceset="FUSE" device="" package3d_urn="urn:adsk.eagle:package:26650/1"/>
-<part name="F2" library="special" library_urn="urn:adsk.eagle:library:367" deviceset="FUSE" device="" package3d_urn="urn:adsk.eagle:package:26650/1"/>
-<part name="F3" library="special" library_urn="urn:adsk.eagle:library:367" deviceset="FUSE" device="" package3d_urn="urn:adsk.eagle:package:26650/1"/>
+<part name="F1" library="special" library_urn="urn:adsk.eagle:library:367" deviceset="FUSE" device="" package3d_urn="urn:adsk.eagle:package:26650/1" value="1A"/>
+<part name="F2" library="special" library_urn="urn:adsk.eagle:library:367" deviceset="FUSE" device="" package3d_urn="urn:adsk.eagle:package:26650/1" value="1A"/>
+<part name="F3" library="special" library_urn="urn:adsk.eagle:library:367" deviceset="FUSE" device="" package3d_urn="urn:adsk.eagle:package:26650/1" value="1A"/>
 <part name="X2" library="con-phoenix-508" library_urn="urn:adsk.eagle:library:176" deviceset="MKDSN1,5/2-5,08" device="" package3d_urn="urn:adsk.eagle:package:9630/1"/>
 <part name="FRAME5" library="frames" library_urn="urn:adsk.eagle:library:229" deviceset="DINA4_L" device=""/>
