File: LSDTivSegG1/regelschaltplan_e7.brd (EAGLE design)
At the start: 160 x 100 mm, 89 parts, among them IC1 LF33AB, IC10 LTV844, IC11 LTV844, IC3 MAX232, IC4 MEGA32-P, Q2 BSS101, Q3 BSS101, Q4 BSS101, Q5 BSS101, Q6 BSS101, Q7 BSS101, Q8 BSS101, Q9 BSS101

Commit message: edit optokoppler with hpcl2621
Parts:
- removed IC10, IC11: LTV844, lsd2016:DIL16
- removed Q9: BSS101, transistor-fet:TO92
- removed R28, R29, R30, R31, R32, R33: 10k, rcl:0207/10
- added C20: 1000u, rcl:C025-025X050
- added OK1, OK2, OK3: HCPL2630, optocoupler:DIL08
- added R18: 10K, rcl:0207/7
- added R19, R20, R21, R22, R23: 10k, rcl:0207/10
- C5: value 1000u -> 100n
- Q2, Q3, Q4, Q5, Q6, Q7, Q8: value BSS101 -> BS170; device transistor-fet:TO92 -> transistor-small-signal:SOT54E
- R10: value 10K -> 10k; device rcl:0207/7 -> rcl:0207/10
- R15, R16, R17, R25, R26, R27: value 220 -> 330
- moved R10 241.1 mm to (-43.2, -165.1)
- moved C5 205.7 mm to (-7.62, -157.5)
- moved SJ1 35.6 mm to (127.0, 68.6), turned to 270 degrees
- moved SJ8 35.6 mm to (91.4, 68.6), turned to 270 degrees
- moved SJ2 25.4 mm to (121.9, 68.6), turned to 270 degrees
- moved SJ7 25.4 mm to (96.5, 68.6), turned to 270 degrees
- moved SJ3 15.2 mm to (116.8, 68.6), turned to 270 degrees
- moved SJ6 15.2 mm to (101.6, 68.6), turned to 270 degrees
- moved Q2 10.2 mm to (81.3, 76.2)
- moved Q3 7.62 mm to (88.9, 76.2)
- moved Q4 5.08 mm to (96.5, 76.2)
- moved Q8 5.08 mm to (127.0, 76.2)
- moved SJ4 5.08 mm to (111.8, 68.6), turned to 270 degrees
- moved SJ5 5.08 mm to (106.7, 68.6), turned to 270 degrees
- moved Q5 2.54 mm to (104.1, 76.2)
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Connections:
- removed net N$33: Q5.3, SJ4.1
- removed net N$35: Q3.3, SJ2.1
- removed net N$47: C5.1, IC4.21, R10.1
- removed net VCC: IC3.16
- new net MOTOR_PWM_RST: LEISTUNG.4
- new net N$12: C20.1, IC4.40, R18.1
- new net N$13: LED6.A, Q8.S
- new net NS1234: C9.-, IC3.5
- net +3V3: now also Q4.G; no longer Q9.2
- net +5V: now also C5.1, IC3.16, R15.1, R16.1, R17.1, R23.2, R26.1, R27.1; no longer C10.-, Q8.2, R31.1
- net 5V_LST: now also OK1.8, OK2.8, OK3.8, R10.2, R19.2, R20.2, R21.2, R22.2, R25.1; no longer R28.1, R29.1, R30.1, R32.1, R33.1
- net BAT_-: now also OK1.5, OK2.5, OK3.5; no longer IC10.11, IC10.13, IC10.15, IC10.8, IC11.13, IC11.15
- net BAT_PWM_CTL: now also Q5.G, R18.2, R23.1; no longer IC10.10, Q7.2, R10.2, R31.2
- net BAT_PWM_LST: now also OK2.3; no longer R25.1
- net DIRL_CTL: now also OK1.2, Q8.G; no longer Q4.2, R15.1
- net DIRL_LST: now also OK1.7, R10.1; no longer IC10.16, R28.2
- net DIRR_CTL: now also OK1.3, Q6.G; no longer Q5.2, R16.1
- net DIRR_LST: now also OK1.6, R19.1; no longer IC10.14, R29.2
- net ENABLE_CTL: now also OK2.2, Q3.G; no longer IC4.26, Q6.2, R17.1
- net ENABLE_LST: now also OK2.7, R20.1; no longer IC10.12, R30.2
- net GND: now also C10.-, C20.2; no longer IC10.2, IC10.4, IC10.6, IC10.9, IC11.2, IC11.4
- net MOTOR_PWM_LST: no longer LEISTUNG.4
- net MOTOR_PWM_L_CTL: now also OK3.2, Q2.G; no longer Q2.2, R26.1
- net MOTOR_PWM_L_LST: now also OK3.7, R21.1; no longer IC11.16, R32.2
- net MOTOR_PWM_R_CTL: now also OK3.3, Q7.G; no longer Q3.2, R27.1
- net MOTOR_PWM_R_LST: now also R22.1; no longer IC11.14, R33.2
- net N$19: now also LED8.A, Q3.S; no longer Q9.3, SJ8.1
- net N$20: now also SJ7.1; no longer Q8.1
- net N$21: now also Q5.S; no longer Q7.1
- net N$22: now also Q4.D, SJ8.1; no longer LED11.A, Q9.1
- net N$23: now also Q6.S; no longer Q5.1
- net N$24: now also Q7.S; no longer Q3.1
- net N$25: now also Q7.D, SJ2.1; no longer LED6.A, Q4.1
- net N$26: now also Q2.S; no longer Q2.1
- net N$27: now also LED11.A, Q4.S; no longer LED8.A, Q6.1
- net N$30: now also Q6.D, SJ4.1; no longer Q8.3, SJ7.1
- net N$31: now also Q5.D; no longer Q7.3
- net N$32: now also Q3.D; no longer Q6.3
- net N$34: now also Q8.D; no longer Q4.3
- net N$36: now also OK1.1; no longer IC10.1
- net N$37: now also OK1.4; no longer IC10.3
- net N$38: now also OK2.1; no longer IC10.5
- net N$39: now also OK2.4; no longer IC10.7
- net N$4: now also Q2.D; no longer Q2.3
- net N$40: now also OK3.4; no longer IC11.3
- net N$41: now also OK3.1; no longer IC11.1
- net RS232RX_CON: now also X1.2; no longer X1.3
- net RS232TX_CON: now also X1.3; no longer X1.4
- net TXD: no longer C9.-, IC3.5

Commit message: worked on regelschaltplan
Parts:
- C20: device rcl:C025-025X050 -> rcl:E2,5-6E
- moved R23 243.1 mm to (63.5, 27.9), turned to 270 degrees
- moved C5 238.5 mm to (45.7, 74.9), turned to 180 degrees
- moved R19 237.2 mm to (15.2, 59.7), turned to 180 degrees
- moved R22 229.2 mm to (17.8, 35.6), turned to 180 degrees
- moved R10 228.6 mm to (15.2, 55.9), turned to 180 degrees
- moved R20 227.3 mm to (15.2, 44.5), turned to 180 degrees
- moved R21 219.5 mm to (17.8, 30.5), turned to 180 degrees
- moved OK1 216.3 mm to (30.5, 58.4), turned to 90 degrees
- moved OK2 207.3 mm to (30.5, 45.7), turned to 90 degrees
- moved OK3 199.5 mm to (30.5, 33.0), turned to 90 degrees
- moved R18 171.5 mm to (73.7, 53.3), turned to 180 degrees
- moved JP2 161.6 mm to (15.2, 78.7), turned to 270 degrees
- moved C4 103.4 mm to (109.2, 55.9), turned to 90 degrees
- moved R16 103.1 mm to (44.5, 62.2), turned to 180 degrees
- moved C18 102.3 mm to (43.2, 16.5), turned to 180 degrees
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Connections:
- removed net MOTOR_PWM_LST: LEISTUNG.2
- removed net MOTOR_PWM_RST: LEISTUNG.4
- removed net NC: LEISTUNG.10
- net +24V: now also LEISTUNG.10
- net BAT_PWM_CTL: now also OK2.6
- net GND: now also C20.-; no longer C20.2
- net MOTOR_PWM_L_LST: now also LEISTUNG.2
- net MOTOR_PWM_R_LST: now also LEISTUNG.4, OK3.6
- net N$12: now also C20.+; no longer C20.1
