File: LSDTivSegG1/regelschaltplan_e7.sch (EAGLE design)
At the start: 88 parts, among them IC1 LF33AB, IC10 LTV844, IC11 LTV844, IC3 MAX232, IC4 MEGA32-P, Q2 BSS101, Q3 BSS101, Q4 BSS101, Q5 BSS101, Q6 BSS101, Q7 BSS101, Q8 BSS101, Q9 BSS101

Commit message: edit optokoppler with hpcl2621
Parts:
- removed IC10, IC11: LTV844, lsd2016:LTV844
- removed Q9: BSS101, transistor-fet:BSS101
- removed R28, R29, R30, R31, R32, R33: 10k, rcl:R-EU_0207/10
- added C20: 1000u, rcl:C-EU025-025X050
- added OK1, OK2, OK3: HCPL2630, optocoupler:HCPL2630
- added R18: 10K, rcl:R-EU_0207/7
- added R19, R20, R21, R22, R23: 10k, rcl:R-EU_0207/10
- C5: value 1000u -> 100n
- Q2, Q3, Q4, Q5, Q6, Q7, Q8: value BSS101 -> BS170; device transistor-fet:BSS101 -> transistor-small-signal:BS170
- R10: value 10K -> 10k; device rcl:R-EU_0207/7 -> rcl:R-EU_0207/10
- R15, R16, R17, R25, R26, R27: value 220 -> 330
Connections:
- removed net N$33: Q5.D, SJ4.1
- removed net N$35: Q3.D, SJ2.1
- removed net N$47: C5.1, IC4.(OC2)PD7, R10.1
- new net MOTOR_PWM_RST: LEISTUNG-4.S
- new net N$12: C20.1, IC4.(ADC0)PA0, R18.1
- new net N$13: LED6.A, Q8.S
- new net NS1234: C9.-, IC3G$1.C2-
- net +3V3: now also Q4.G; no longer Q9.G
- net +5V: now also C5.1, IC3P.VCC, R15.1, R16.1, R17.1, R23.2, R26.1, R27.1; no longer C10.-, Q8.G, R31.1
- net 5V_LST: now also OK1A.VCC, OK2A.VCC, OK3A.VCC, R10.2, R19.2, R20.2, R21.2, R22.2, R25.1; no longer R28.1, R29.1, R30.1, R32.1, R33.1
- net BAT_-: now also OK1A.GND, OK2A.GND, OK3A.GND; no longer IC10G$1.EMIT, IC10G$2.EMIT, IC10G$3.EMIT, IC10G$4.C, IC11G$1.EMIT, IC11G$2.EMIT
- net BAT_PWM_CTL: now also Q5.G, R18.2, R23.1; no longer IC10G$4.COL, Q7.G, R10.2, R31.2
- net BAT_PWM_LST: now also OK2B.C2; no longer R25.1
- net DIRL_CTL: now also OK1A.C1, Q8.G; no longer Q4.G, R15.1
- net DIRL_LST: now also OK1A.VO1, R10.1; no longer IC10G$1.COL, R28.2
- net DIRR_CTL: now also OK1B.C2, Q6.G; no longer Q5.G, R16.1
- net DIRR_LST: now also OK1B.VO2, R19.1; no longer IC10G$2.COL, R29.2
- net ENABLE_CTL: now also OK2A.C1, Q3.G; no longer IC4.(TDO)PC4, Q6.G, R17.1
- net ENABLE_LST: now also OK2A.VO1, R20.1; no longer IC10G$3.COL, R30.2
- net GND: now also C10.-, C20.2, IC3P.GND; no longer IC10G$1.C, IC10G$2.C, IC10G$3.C, IC10G$4.EMIT, IC11G$1.C, IC11G$2.C
- net MOTOR_PWM_LST: no longer LEISTUNG-4.S
- net MOTOR_PWM_L_CTL: now also OK3A.C1; no longer R26.1
- net MOTOR_PWM_L_LST: now also OK3A.VO1, R21.1; no longer IC11G$1.COL, R32.2
- net MOTOR_PWM_R_CTL: now also OK3B.C2, Q7.G; no longer Q3.G, R27.1
- net MOTOR_PWM_R_LST: now also R22.1; no longer IC11G$2.COL, R33.2
- net N$19: now also LED8.A, Q3.S; no longer Q9.D, SJ8.1
- net N$20: now also SJ7.1; no longer Q8.S
- net N$21: now also Q5.S; no longer Q7.S
- net N$22: now also Q4.D, SJ8.1; no longer LED11.A, Q9.S
- net N$23: now also Q6.S; no longer Q5.S
- net N$24: now also Q7.S; no longer Q3.S
- net N$25: now also Q7.D, SJ2.1; no longer LED6.A, Q4.S
- net N$27: now also LED11.A, Q4.S; no longer LED8.A, Q6.S
- net N$30: now also Q6.D, SJ4.1; no longer Q8.D, SJ7.1
- net N$31: now also Q5.D; no longer Q7.D
- net N$32: now also Q3.D; no longer Q6.D
- net N$34: now also Q8.D; no longer Q4.D
- net N$36: now also OK1A.A1; no longer IC10G$1.A
- net N$37: now also OK1B.A2; no longer IC10G$2.A
- net N$38: now also OK2A.A1; no longer IC10G$3.A
- net N$39: now also OK2B.A2; no longer IC10G$4.A
- net N$40: now also OK3B.A2; no longer IC11G$2.A
- net N$41: now also OK3A.A1; no longer IC11G$1.A
- net RS232RX_CON: now also X1.2; no longer X1.3
- net RS232TX_CON: now also X1.3; no longer X1.4
- net TXD: no longer C9.-, IC3G$1.C2-

Commit message: worked on regelschaltplan
Parts:
- C20: device rcl:C-EU025-025X050 -> rcl:CPOL-USE2,5-6E
Connections:
- removed net MOTOR_PWM_LST: LEISTUNG-2.S
- removed net MOTOR_PWM_RST: LEISTUNG-4.S
- removed net NC: LEISTUNG-10.S
- net +24V: now also LEISTUNG-10.S
- net BAT_PWM_CTL: now also OK2B.VO2
- net GND: now also C20.-; no longer C20.2
- net MOTOR_PWM_L_LST: now also LEISTUNG-2.S
- net MOTOR_PWM_R_LST: now also LEISTUNG-4.S, OK3B.VO2
- net N$12: now also C20.+; no longer C20.1
