File: LSDTivSegG1/leistung.brd (EAGLE design)
At the start: 160 x 100 mm, 87 parts, among them IC1 LM 2576 T5,0, IC2 IR2184D, IC3 IR2184D, IC4 4081N, IC5 4069N, IC6 LM 2576 T15, IC7 IR2184D, IC8 IR2184D, IC9 TINY13-20PU, Q1 IRFB3077, Q10 IRFB3077, Q11 IRFB3077, Q12 IRFB3077, Q2 IRFB3077, Q3 IRFB3077, Q4 IRFB3077, Q9 IRFB3077, X1 057-010-1, X2 MKDSN1,5/2-5,08

Commit message: layouted H-Bridges
Parts:
- L1, L2: device rcl:0204/5 -> rcl:0207/10
- moved C20 194.0 mm to (25.4, 29.2), turned to 180 degrees
- moved C19 182.1 mm to (26.7, 10.2)
- moved C11 181.6 mm to (10.2, 19.1), turned to 180 degrees
- moved C4 147.6 mm to (88.9, 36.8), turned to 180 degrees
- moved C10 140.9 mm to (229.9, -47.0)
- moved C16 140.9 mm to (237.5, -44.5)
- moved R10 140.9 mm to (251.5, -50.8)
- moved C17 140.9 mm to (231.1, -31.8)
- moved C18 140.9 mm to (231.1, -14.0)
- moved IC4 140.9 mm to (242.6, -31.8)
- moved IC5 140.9 mm to (242.6, -14.0)
- moved IC9 140.9 mm to (238.8, -50.8)
- moved R16 140.9 mm to (259.1, -49.5)
- moved R9 140.9 mm to (262.9, -49.5)
- moved C5 135.1 mm to (88.9, 14.0), turned to 180 degrees
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Routing:
- net MOTOR_L_-: track 7.62 -> 112.0 mm
- net BAT_+: track 7.62 -> 85.1 mm
- net MOTOR_R_-: track 7.62 -> 77.7 mm
- net MOTOR_R_+: track 7.62 -> 76.6 mm
- net MOTOR_L_+: track 28.0 -> 89.7 mm
- net ENABLE: track 9.42 -> 36.5 mm
- net N$7: track 0.00 -> 11.7 mm
- net N$30: track 0.00 -> 11.7 mm
- net N$31: track 0.00 -> 11.7 mm
- net VB2: track 0.00 -> 9.94 mm
- net VB3: track 0.00 -> 9.94 mm
- net VB4: track 0.00 -> 9.94 mm
- net IN_L: track 6.88 -> 16.5 mm
- net N$32: track 0.00 -> 6.88 mm
- net N$13: track 0.00 -> 6.88 mm
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- added copper zone on layer 16, net BAT_+
- removed copper zone on layer 1, net BAT_+
Other:
- board size 160 x 100 mm -> 150 x 100 mm

Commit message: finalized board
Parts:
- removed IC1: LM 2576 T5,0, LM2576:TO-220-5_IN-LINE
- removed IC6: LM 2576 T15, LM2576:TO-220-5_IN-LINE
- added IC10: LM 2576 T15, LM2576:TO220-5_STAGGERED
- added IC11: LM 2576 T5.0, LM2576:TO220-5_STAGGERED
- moved IC4 177.2 mm to (96.5, 68.6), turned to 270 degrees
- moved C17 174.2 mm to (96.5, 78.7), turned to 180 degrees
- moved C9 160.6 mm to (141.6, 39.0)
- moved D8 159.0 mm to (127.0, 45.7)
- moved R16 154.9 mm to (125.7, 29.2), turned to 180 degrees
- moved IC5 153.4 mm to (94.0, 24.1), turned to 180 degrees
- moved L2 146.6 mm to (124.5, 41.9)
- moved R9 146.0 mm to (130.8, 12.7), turned to 0 degrees
- moved C8 134.7 mm to (118.1, 33.0), turned to 90 degrees
- moved IC9 133.9 mm to (127.0, 22.9), turned to 90 degrees
- moved R10 132.5 mm to (139.7, 20.3)
- moved C18 131.4 mm to (105.4, 24.1)
- moved R15 128.2 mm to (133.3, 35.6), turned to 270 degrees
- moved LED2 123.6 mm to (137.2, 30.5)
- moved C10 120.2 mm to (127.0, 15.2), turned to 180 degrees
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Connections:
- net +15V: now also IC10.P$4; no longer IC6.P$4
- net +24V: now also IC10.P$1, IC11.P$1; no longer IC1.P$1, IC6.P$1
- net +5V: now also IC11.P$4; no longer IC1.P$4
- net GND: now also IC10.P$3, IC10.P$5, IC11.P$3, IC11.P$5; no longer IC1.P$3, IC1.P$5, IC6.P$3, IC6.P$5
- net N$1: now also IC11.P$2; no longer IC1.P$2
- net N$4: now also IC10.P$2; no longer IC6.P$2
Routing:
- net +5V: track 0.00 -> 211.0 mm, vias 0 -> 1
- net GND: track 0.00 -> 193.0 mm, vias 0 -> 7
- net +15V: track 29.6 -> 209.0 mm, vias 0 -> 2
- net ENABLE: track 36.5 -> 162.1 mm, vias 0 -> 2
- net +24V: track 0.00 -> 124.0 mm, vias 0 -> 3
- net MOTOR_PWM_L: track 0.00 -> 94.4 mm, vias 0 -> 2
- net MOTOR_PWM_R: track 0.00 -> 94.0 mm, vias 0 -> 2
- net DIRR: track 0.00 -> 84.1 mm, vias 0 -> 4
- net DIRL: track 0.00 -> 79.0 mm, vias 0 -> 2
- net IN_L_INVD: track 0.00 -> 68.1 mm, vias 0 -> 2
- net DIRL_INV: track 0.00 -> 60.9 mm, vias 0 -> 2
- net MOTOR_R_-: track 77.7 -> 137.3 mm, vias 0 -> 2
- net MOTOR_R_+: track 76.6 -> 132.4 mm, vias 0 -> 3
- net BAT_PWM: track 0.00 -> 50.4 mm, vias 0 -> 2
- net IN_R_INVD: track 0.00 -> 47.5 mm, vias 0 -> 2
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